File: Symbiote-Prototype1/Symbiote.kicad_sch (KiCad schematic)
At the start: 27 parts, among them J1 Micro_SD_Card, SW1 SW_DIP_x01, SW2 SW_DIP_x01, U1 STM32F401RETx, U2 ADS1263IPW, U3 ADS1263IPW, U4 ADS1263IPW, U5 RFD22301, U6 LIS3DH, Y1 8m

Commit message: Connect ADC to different SPI
Connections:
- net MISO: no longer U3.13 (DOUT/DRDY), U4.13 (DOUT/DRDY)
- net MOSI: no longer U3.12 (DIN), U4.12 (DIN)
- net MISO2: now reaches U1.10 (PC2)
- net MISO2: now also U3.13 (DOUT/DRDY)
- net MOSI2: now reaches U1.36 (PB15)
- net MOSI2: now also U3.12 (DIN)
- net MISO3: now reaches U1.52 (PC11)
- net MISO3: now also U4.13 (DOUT/DRDY)
- net MOSI3: now reaches U1.53 (PC12)
- net MOSI3: now also U4.12 (DIN)
Changed lines of the file:
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@@
+	(wire
+		(pts
+			(xy 137.16 284.48) (xy 157.48 284.48)
+		)
+		(stroke
+			(width 0)
+			(type default)
+		)
+	)
 	(wire
 		(pts
@@
 	(wire
 		(pts
+			(xy 137.16 281.94) (xy 157.48 281.94)
+		)
+		(stroke
+			(width 0)
+			(type default)
+		)
+	)
+	(wire
+		(pts
 			(xy 638.81 83.82) (xy 642.62 83.82)
 		)
@@
 	(wire
 		(pts
+			(xy 135.89 259.08) (xy 157.48 259.08)
+		)
+		(stroke
+			(width 0)
+			(type default)
+		)
+	)
+	(wire
+		(pts
 			(xy 387.35 186.69) (xy 393.7 186.69)
 		)
@@
 		(pts
 			(xy 151.13 222.25) (xy 151.13 226.06)
+		)
+		(stroke
+			(width 0)
+			(type default)
+		)
+	)
+	(wire
+		(pts
+			(xy 190.5 304.8) (xy 218.44 304.8)
 		)
 		(stroke
@@
 		)
 	)
+	(label "MOSI3"
+		(at 137.16 284.48 0)
+		(fields_autoplaced yes)
+		(effects
+			(font
+				(size 1.27 1.27)
+			)
+			(justify left bottom)
+		)
+	)
+	(label "MISO3"
+		(at 137.16 281.94 0)
+		(fields_autoplaced yes)
+		(effects
+			(font
+				(size 1.27 1.27)
+			)
+			(justify left bottom)
+		)
+	)
 	(label "SCL"
 		(at 321.31 97.79 0)
@@
 		)
 	)
-	(label "MOSI"
+	(label "MOSI2"
 		(at 330.2 219.71 0)
 		(fields_autoplaced yes)
@@
 		)
 	)
-	(label "MISO"
+	(label "MISO2"
 		(at 387.35 191.77 0)
 		(fields_autoplaced yes)
@@
 		)
 	)
-	(label "MOSI"
+	(label "MOSI3"
 		(at 328.93 341.63 0)
 		(fields_autoplaced yes)
@@
 		)
 	)
-	(label "MISO"
+	(label "MISO3"
 		(at 387.35 313.69 0)
+		(fields_autoplaced yes)
+		(effects
+			(font
+				(size 1.27 1.27)
+			)
+			(justify left bottom)
+		)
+	)
+	(label "MISO2"
+		(at 135.89 259.08 0)
 		(fields_autoplaced yes)
 		(effects
@@
 		(fields_autoplaced yes)
 		(effects
+			(font
+				(size 1.27 1.27)
+			)
+			(justify left bottom)
+		)
+	)
+	(label "MOSI2"
+		(at 218.44 304.8 0)
+		(fields_autoplaced yes)
+		(effects
